Commit message: Updated robot_arm urdf

File: simulation/urdf/robot_arm.urdf (robot description, URDF)
Before this commit: robot robotic_arm, 2 links, 1 joints
Links:
- removed link link1
- added link arm1, mass 1; collision box size=0.1 1.1 0.1; visual box size=0.1 1.1 0.1
- added link arm2, mass 1; collision box size=0.1 0.9 0.1; visual box size=0.1 0.9 0.1
- added link world
- link base_link: mass None -> 1; geometry collision cylinder length=1.0 radius=0.1; visual cylinder length=1.0 radius=0.1
Joints:
- removed joint joint1
- added joint rotation0: type revolute, parent world, child base_link, origin xyz=0 0 0 rpy=0 0 0, axis 0 0 1, limit lower=-3.14 upper=3.14 effort=100 velocity=10
- added joint rotation1: type revolute, parent base_link, child arm1, origin xyz=0 0 1.0 rpy=0 1.57075 0, axis 0 0 1, limit lower=-3.14 upper=3.14 effort=100 velocity=10
- added joint rotation2: type revolute, parent arm1, child arm2, origin xyz=0 -1 0.1 rpy=0 0 0, axis 0 0 1, limit lower=-3.00 upper=3.00 effort=1000 velocity=1000
